File: Circuits/P_SUPPLY.sch (KiCad schematic (older format))
At the start: 28 parts, among them P1 127VAC, P2 ON/OFF SW, P3 SYMMETRIC 8V, P4 +5V OUTPUT, T1 127:12, U1 LM7808CT, U2 LM7805CT, U3 LM7908CT

Commit message: ADD: Complete Power Supply SCH+PCB
Parts:
- P3: value SYMMETRIC 8V -> SYMMETRIC 8V OUT; footprint (none) -> Connectors:bornier3
- P4: footprint (none) -> Connectors:bornier2
- T1: footprint (none) -> Transformers_THT:12V_transformer-3T
- U1, U3: footprint TO-220 -> Power_Integrations:TO-220
- U2: footprint TO_SOT_Packages_THT:TO-220_Vertical -> Power_Integrations:TO-220
Changed lines of the file:
@@
 LIBS:Zilog
 LIBS:P_SUPPLY-cache
-LIBS:ElectricKettle-cache
 EELAYER 25 0
 EELAYER END
@@
 F 0 "U2" H 2350 4300 50  0000 C CNN
 F 1 "LM7805CT" H 2550 4300 50  0000 L CNN
-F 2 "TO_SOT_Packages_THT:TO-220_Vertical" H 2550 4200 50  0001 C CIN
+F 2 "Power_Integrations:TO-220" H 2550 4200 50  0001 C CIN
 F 3 "" H 2550 4100 50  0000 C CNN
 	1    2550 4100
@@
 F 0 "U1" H 1350 2900 50  0000 C CNN
 F 1 "LM7808CT" H 1450 2900 50  0000 L CNN
-F 2 "TO-220" H 1550 2800 50  0000 C CIN
+F 2 "Power_Integrations:TO-220" H 1550 2800 50  0000 C CIN
 F 3 "" H 1550 2700 50  0000 C CNN
 	1    1550 2700
@@
 F 0 "T1" H 2600 1150 50  0000 C CNN
 F 1 "127:12" H 2600 1750 50  0000 C CNN
-F 2 "" H 2600 1450 50  0000 C CNN
+F 2 "Transformers_THT:12V_transformer-3T" H 2600 1450 50  0001 C CNN
 F 3 "" H 2600 1450 50  0000 C CNN
 	1    2600 1450
@@
 F 0 "U3" H 3350 2500 50  0000 C CNN
 F 1 "LM7908CT" H 3450 2500 50  0000 L CNN
-F 2 "TO-220" H 3550 2600 50  0000 C CIN
+F 2 "Power_Integrations:TO-220" H 3550 2600 50  0000 C CIN
 F 3 "" H 3550 2700 50  0000 C CNN
 	1    3550 2700
@@
 F 0 "P4" H 3700 5550 50  0000 C CNN
 F 1 "+5V OUTPUT" V 3800 5400 50  0000 C CNN
-F 2 "" H 3700 5400 50  0000 C CNN
+F 2 "Connectors:bornier2" H 3700 5400 50  0001 C CNN
 F 3 "" H 3700 5400 50  0000 C CNN
 	1    3700 5400
@@
 P 2900 5450
 F 0 "P3" H 2900 5650 50  0000 C CNN
-F 1 "SYMMETRIC 8V" V 3000 5450 50  0000 C CNN
-F 2 "" H 2900 5450 50  0000 C CNN
+F 1 "SYMMETRIC 8V OUT" V 3000 5450 50  0000 C CNN
+F 2 "Connectors:bornier3" H 2900 5450 50  0001 C CNN
 F 3 "" H 2900 5450 50  0000 C CNN
 	1    2900 5450
