File: Circuits/I_SOURCE/I_SOURCE.kicad_pcb (KiCad board)
At the start: 2 copper layers, 74.8 x 50 mm, 34 parts, among them P1 POWER, P2 I_SELECT, P3 OUTPUT, Q1 TIP127, U1 CA3140, U2 LM393

Commit message: ADD: Complete Current Source SCH+PCB w/ Gerbers
Parts:
- moved Q1 119.1 mm to (100.0, 165.8)
- moved R7 117.8 mm to (102.5, 185.3)
- moved C1 117.8 mm to (78.0, 169.2)
- moved C2 117.8 mm to (111.0, 165.2)
- moved C3 117.8 mm to (116.3, 145.1)
- moved C4 117.8 mm to (78.0, 177.2)
- moved C5 117.8 mm to (102.5, 175.5)
- moved C6 117.8 mm to (126.8, 145.0)
- moved C7 117.8 mm to (132.8, 151.3)
- moved D1 117.8 mm to (129.9, 179.9)
- moved G*** 117.8 mm to (142.2, 186.0)
- moved G*** 117.8 mm to (142.2, 177.0)
- moved P1 117.8 mm to (94.2, 148.8)
- moved P3 117.8 mm to (113.8, 182.1)
- moved R1 117.8 mm to (115.8, 159.8)
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Routing:
- net +8V: track 186.1 -> 163.3 mm
- net -8V: track 73.2 -> 76.0 mm
- net I_OUT: track 42.2 -> 40.6 mm
- net Net-(P2-Pad2): track 36.6 -> 35.4 mm
- net Net-(P2-Pad1): track 2.80 -> 4.02 mm
- net Net-(P2-Pad3): track 10.5 -> 11.7 mm
- net Net-(Q1-Pad1): track 4.77 -> 5.74 mm
- net Net-(R1-Pad2): track 11.1 -> 11.7 mm
Other:
- board text added: "Designed by Alisson Claudino"
- board text added: "I SELECT(A)"
- board text removed: "Current Select"

Commit message: ADD: Current Source fabrication files
Parts:
- moved REF** 2.12 mm to (76.8, 146.0)
- moved G*** 2.02 mm to (140.2, 185.8)
- moved REF** 1.41 mm to (144.0, 145.5)
- moved REF** 1.41 mm to (144.0, 188.5)
- moved REF** 1.41 mm to (76.2, 188.5)
Changed lines of the file:
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@@
     (visible_elements FFFFFF7F)
     (pcbplotparams
-      (layerselection 0x00020_00000000)
+      (layerselection 0x01000_80000001)
       (usegerberextensions false)
       (excludeedgelayer true)
@@
       (viasonmask false)
       (mode 1)
-      (useauxorigin false)
+      (useauxorigin true)
       (hpglpennumber 1)
       (hpglpenspeed 20)
@@
       (padsonsilk true)
       (subtractmaskfromsilk false)
-      (outputformat 4)
+      (outputformat 1)
       (mirror false)
-      (drillshape 1)
+      (drillshape 0)
       (scaleselection 1)
-      (outputdirectory /home/alissomc/SADAMAP/Circuits/I_SOURCE/))
+      (outputdirectory "/home/alissomc/SADAMAP/Circuits/I_SOURCE/Fabrication Files/Gerbers/"))
   )
   (net 0 "")
@@
   )
   (module Mounting_Holes:MountingHole_2.2mm_M2 (layer F.Cu)
-    (at 145 144.5)
+    (at 144 145.5)
     (descr "Mounting Hole 2.2mm, no annular, M2")
     (tags "mounting hole 2.2mm no annular m2")
@@
   )
   (module Mounting_Holes:MountingHole_2.2mm_M2 (layer F.Cu)
-    (at 145 189.5)
+    (at 144 188.5)
     (descr "Mounting Hole 2.2mm, no annular, M2")
     (tags "mounting hole 2.2mm no annular m2")
@@
   )
   (module Mounting_Holes:MountingHole_2.2mm_M2 (layer F.Cu)
-    (at 75.25 189.5)
+    (at 76.25 188.5)
     (descr "Mounting Hole 2.2mm, no annular, M2")
     (tags "mounting hole 2.2mm no annular m2")
@@
   )
   (module Symbols:cta (layer F.Cu)
-    (at 142.25 186 90)
+    (at 140.25 185.75 90)
     (fp_text reference G*** (at 0 0 90) (layer F.SilkS) hide
       (effects (font (thickness 0.3)))
@@
   )
   (module Mounting_Holes:MountingHole_2.2mm_M2 (layer F.Cu)
-    (at 75.25 144.5)
+    (at 76.75 146)
     (descr "Mounting Hole 2.2mm, no annular, M2")
     (tags "mounting hole 2.2mm no annular m2")
