File: Circuits/V_AMP/V_AMP.sch (KiCad schematic (older format))
At the start: 41 parts, among them P1 INPUT, P2 GAIN_ADJ, P3 OUTPUT (0-5V), P4 POWER, U1 OPA277, U2 LM393, U3 OPA277

Commit message: ADD: Complete Current Source SCH+PCB w/ Gerbers
Parts:
- RV1: footprint Potentiometers:Potentiometer_Alps_RK163_Single_Vertical -> Potentiometers:Potentiometer_Trimmer_Bourns_3296X
Changed lines of the file:
@@
 F 0 "RV1" H 5200 3870 50  0000 C CNN
 F 1 "50k" H 5200 3950 50  0000 C CNN
-F 2 "Potentiometers:Potentiometer_Alps_RK163_Single_Vertical" H 5200 3950 50  0001 C CNN
+F 2 "Potentiometers:Potentiometer_Trimmer_Bourns_3296X" H 5200 3950 50  0001 C CNN
 F 3 "" H 5200 3950 50  0000 C CNN
 	1    5200 3950

Commit message: EDIT: V_AMP is a PGA now
Parts:
- removed C7, C9: 220n, Capacitors_THT:C_Rect_L7.0mm_W2.5mm_P5.00mm, symbol C
- removed C8: 100n, Capacitors_THT:C_Rect_L7.0mm_W2.5mm_P5.00mm, symbol C_Small
- removed D4: 5V1, Diodes_THT:D_DO-41_SOD81_P7.62mm_Horizontal, symbol ZENERsmall
- removed P2: GAIN_ADJ, w_pin_strip:pin_strip_2mm_2, symbol CONN_01X02
- removed P3: OUTPUT (0-5V), Connectors:bnc-ci, symbol BNC
- removed R10: 10k, w_pth_resistors:RC03, symbol R
- removed R11: RX, w_pth_resistors:RC03, symbol R
- removed R12: 2k7, w_pth_resistors:RC03, symbol R
- removed R13: 27k, w_pth_resistors:RC03, symbol R
- removed R14: 100, w_pth_resistors:RC03, symbol R
- removed R4: 20k, w_pth_resistors:RC03, symbol R
- removed R5: 180k, w_pth_resistors:RC03, symbol R
- removed RV1: 50k, Potentiometers:Potentiometer_Trimmer_Bourns_3296X, symbol POT
- removed U3: OPA277, Housings_DIP:DIP-8_W7.62mm_Socket_LongPads, symbol OPA177
- added C7, C8: 100n, symbol Device:C_Small
- added C9: 10u, symbol Device:CP1_Small
- added D4, D6: 5V1, symbol device:ZENERsmall
- added P2: BNC, symbol conn:BNC
- added P3: CONTROL_IN, symbol conn:CONN_01X05
- added R10, R11, R4, R5: 100k, w_pth_resistors:RC03, symbol V_AMP-rescue:R
- added R12, R24: 2k7, w_pth_resistors:RC03, symbol V_AMP-rescue:R
- added R13: 10k, w_pth_resistors:RC03, symbol V_AMP-rescue:R
- added R14: 1k, w_pth_resistors:RC03, symbol V_AMP-rescue:R
- added R18, R19: 750, w_pth_resistors:RC03, symbol V_AMP-rescue:R
- added R20, R21: 150, w_pth_resistors:RC03, symbol V_AMP-rescue:R
- added R22: 820, symbol Device:R
- added R23: DNP, w_pth_resistors:RC03, symbol V_AMP-rescue:R
- added RV1: 2k, symbol Device:POT
- added U3: DG412xJ, Package_DIP:DIP-16_W7.62mm, symbol Analog_Switch:DG412xJ
- C1, C2: symbol C -> V_AMP-rescue:C
- C10, C11: symbol CP_Small -> V_AMP-rescue:CP_Small
- C3, C4, C5, C6: symbol C_Small -> V_AMP-rescue:C_Small
- D1, D2: symbol ZENERsmall -> V_AMP-rescue:ZENERsmall
- D3: symbol D_Small -> V_AMP-rescue:D_Small
- D5: symbol LED -> V_AMP-rescue:LED
- P1: symbol BNC -> V_AMP-rescue:BNC
- P4: symbol CONN_01X03 -> V_AMP-rescue:CONN_01X03
- R1, R15, R16, R17, R2, R3, R6, R7, R8, R9: symbol R -> V_AMP-rescue:R
- U1: symbol OPA177 -> V_AMP-rescue:OPA177
- U2: symbol LM393 -> V_AMP-rescue:LM393
Connections:
- net OUT2 is gone; now on net OUT1: R8.2
- net +8V: now also U2.8 (V+), C8.2, R22.2, U3.13 (V+)
- net -8V: now also U2.4 (V-), C7.1, U3.4 (V-)
- net GND: now also C7.2, C8.1, C9.2, D4.2 (A), D6.2 (A), P2.2 (Ext), P3.1 (P1), R10.1, R11.1, R19.1, R21.1, R23.1, R4.1, R5.1, U3.5 (GND)
- net OUT1: now also R12.1, R24.2, RV1.3
- net IN1: now reaches C1.1, R3.1, U1.3 (NON)
- net IN1: now also R23.2
- net at C2.2, U1.2 (INVERTING): now also U3.11, U3.14, U3.3, U3.7
- new net: R12.2, U3.2
- new net: R13.1, R14.2, U3.6
- new net: R14.1, R18.2, R20.2, U3.10
- new net: R18.1, R19.2, R20.1, R21.2, U3.15
- new net: C9.1, D4.1 (K), R22.1, U3.12 (VL)
- new net: R13.2, RV1.1, RV1.2
- new net: D6.1 (K), P2.1 (In), R24.1
- new net b0: P3.5 (P5), R4.2, U3.1
- new net b1: P3.4 (P4), R5.2, U3.8
- new net b2: P3.3 (P3), R10.2, U3.9
- new net b3: P3.2 (P2), R11.2, U3.16
- no-connect marks 9 -> 4
Other:
- note added: "Input Interface"
- note added: "Programmable Gain Amplifier (PGA)\n\n b0 b1 b2 b3 Gain\n 1 0 0 0 1\n 0 1 0 0 10\n 0 0 1 0 50\n 0 0 0 1 100"
- note removed: "1-10x 2nd Stage Amplifier"
- note removed: "10x 1st Stage Amplifier\n"
- moved on the sheet: C1, C10, C11, C2, C3, C4, C5, C6, D1, D2, D3, D5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

Commit message: ADD: V_AMP pcb design
Parts:
- C7, C8: footprint (none) -> Capacitors_THT:C_Rect_L7.0mm_W2.5mm_P5.00mm; symbol Device:C_Small -> device:C_Small
- C9: footprint (none) -> Capacitors_THT:CP_Radial_D5.0mm_P2.50mm; symbol Device:CP1_Small -> device:CP1_Small
- D4: footprint (none) -> Diodes_THT:D_DO-41_SOD81_P7.62mm_Horizontal; symbol device:ZENERsmall -> V_AMP:ZENERsmall
- D6: footprint (none) -> Diodes_THT:D_DO-41_SOD81_P7.62mm_Horizontal; symbol device:ZENERsmall -> V_AMP-rescue:device_ZENERsmall-V_AMP-cache
- P1: footprint Connectors:bnc-ci -> Connect:bornier2
- P2: value BNC -> OUTPUT; footprint (none) -> Connect:bornier2
- P3: footprint (none) -> w_conn_kk100:kk100_22-23-2051
- R22: footprint (none) -> w_pth_resistors:RC03; symbol Device:R -> device:R
- RV1: footprint (none) -> Potentiometers:Potentiometer_Trimmer_Bourns_3296X; symbol Device:POT -> device:POT
- U3: footprint Package_DIP:DIP-16_W7.62mm -> Housings_DIP:DIP-16_W7.62mm_Socket_LongPads; symbol Analog_Switch:DG412xJ -> analog_switches:DG412xJ
Changed lines of the file:
@@
 encoding utf-8
 Sheet 1 1
-Title "1x to 100x Precision Programmable Gain Pre-Amplifier for Generic Sensors "
-Date "2017-12-18"
+Title "1x to 100x Precision Prog. Gain Generic Pre-Amplifier"
+Date "2018-05-22"
 Rev "1"
 Comp "LAPMA/CTA - IF/UFRGS"
@@
 F 0 "P1" H 4800 3450 50  0000 C CNN
 F 1 "INPUT" H 4650 3750 50  0000 C CNN
-F 2 "Connectors:bnc-ci" H 4650 3600 50  0001 C CNN
+F 2 "Connect:bornier2" H 4650 3600 50  0001 C CNN
 F 3 "" H 4650 3600 50  0000 C CNN
 	1    4650 3600
@@
 	5200 3000 5200 3050
 $Comp
-L Analog_Switch:DG412xJ U3
+L analog_switches:DG412xJ U3
 U 1 1 5AD0C3E7
 P 1200 2350
 F 0 "U3" H 1200 2617 50  0000 C CNN
 F 1 "DG412xJ" H 1200 2526 50  0000 C CNN
-F 2 "Package_DIP:DIP-16_W7.62mm" H 1200 2250 50  0001 C CNN
+F 2 "Housings_DIP:DIP-16_W7.62mm_Socket_LongPads" H 1200 2250 50  0001 C CNN
 F 3 "https://datasheets.maximintegrated.com/en/ds/DG411-DG413.pdf" H 1200 2350 50  0001 C CNN
 	1    1200 2350
@@
 $EndComp
 $Comp
-L Analog_Switch:DG412xJ U3
+L analog_switches:DG412xJ U3
 U 2 1 5AD0C511
 P 1200 3200
 F 0 "U3" H 1200 3467 50  0000 C CNN
 F 1 "DG412xJ" H 1200 3376 50  0000 C CNN
-F 2 "Package_DIP:DIP-16_W7.62mm" H 1200 3100 50  0001 C CNN
+F 2 "Housings_DIP:DIP-16_W7.62mm_Socket_LongPads" H 1200 3100 50  0001 C CNN
 F 3 "https://datasheets.maximintegrated.com/en/ds/DG411-DG413.pdf" H 1200 3200 50  0001 C CNN
 	2    1200 3200
@@
 $EndComp
 $Comp
-L Analog_Switch:DG412xJ U3
+L analog_switches:DG412xJ U3
 U 3 1 5AD0C60F
 P 1200 3850
 F 0 "U3" H 1200 4117 50  0000 C CNN
 F 1 "DG412xJ" H 1200 4026 50  0000 C CNN
-F 2 "Package_DIP:DIP-16_W7.62mm" H 1200 3750 50  0001 C CNN
+F 2 "Housings_DIP:DIP-16_W7.62mm_Socket_LongPads" H 1200 3750 50  0001 C CNN
 F 3 "https://datasheets.maximintegrated.com/en/ds/DG411-DG413.pdf" H 1200 3850 50  0001 C CNN
 	3    1200 3850
@@
 $EndComp
 $Comp
-L Analog_Switch:DG412xJ U3
+L analog_switches:DG412xJ U3
 U 4 1 5AD0C691
 P 1200 4500
 F 0 "U3" H 1200 4767 50  0000 C CNN
 F 1 "DG412xJ" H 1200 4676 50  0000 C CNN
-F 2 "Package_DIP:DIP-16_W7.62mm" H 1200 4400 50  0001 C CNN
+F 2 "Housings_DIP:DIP-16_W7.62mm_Socket_LongPads" H 1200 4400 50  0001 C CNN
 F 3 "https://datasheets.maximintegrated.com/en/ds/DG411-DG413.pdf" H 1200 4500 50  0001 C CNN
 	4    1200 4500
@@
 $EndComp
 $Comp
-L Analog_Switch:DG412xJ U3
+L analog_switches:DG412xJ U3
 U 5 1 5AD72EF0
 P 3450 2000
 F 0 "U3" V 3133 2000 50  0000 C CNN
 F 1 "DG412xJ" V 3224 2000 50  0000 C CNN
-F 2 "Package_DIP:DIP-16_W7.62mm" H 3450 1900 50  0001 C CNN
+F 2 "Housings_DIP:DIP-16_W7.62mm_Socket_LongPads" H 3450 1900 50  0001 C CNN
 F 3 "https://datasheets.maximintegrated.com/en/ds/DG411-DG413.pdf" H 3450 2000 50  0001 C CNN
 	5    3450 2000
@@
 $EndComp
 $Comp
-L device:ZENERsmall D4
+L V_AMP:ZENERsmall D4
 U 1 1 5AD7344B
 P 4150 2100
 F 0 "D4" H 4050 2150 50  0000 C CNN
 F 1 "5V1" H 4250 2150 50  0000 C CNN
-F 2 "" H 4150 2100 50  0000 C CNN
+F 2 "Diodes_THT:D_DO-41_SOD81_P7.62mm_Horizontal" H 4150 2100 50  0001 C CNN
 F 3 "" H 4150 2100 50  0000 C CNN
 	1    4150 2100
@@
 $EndComp
 $Comp
-L Device:CP1_Small C9
+L device:CP1_Small C9
 U 1 1 5AD7650A
 P 4150 2250
 F 0 "C9" V 4200 2150 50  0000 C CNN
 F 1 "10u" V 4100 2100 50  0000 C CNN
-F 2 "" H 4150 2250 50  0001 C CNN
+F 2 "Capacitors_THT:CP_Radial_D5.0mm_P2.50mm" H 4150 2250 50  0001 C CNN
 F 3 "~" H 4150 2250 50  0001 C CNN
 	1    4150 2250
@@
 	4000 1950 4050 1950
 $Comp
-L Device:R R22
+L device:R R22
 U 1 1 5AD8742C
 P 4200 2400
 F 0 "R22" V 4150 2550 50  0000 C CNN
 F 1 "820" V 4200 2400 50  0000 C CNN
-F 2 "" V 4130 2400 50  0001 C CNN
+F 2 "w_pth_resistors:RC03" V 4130 2400 50  0001 C CNN
 F 3 "~" H 4200 2400 50  0001 C CNN
 	1    4200 2400
@@
 $EndComp
 $Comp
-L Device:C_Small C8
+L device:C_Small C8
 U 1 1 5AD8FA52
 P 4150 1950
 F 0 "C8" V 4100 1850 50  0000 C CNN
 F 1 "100n" V 4100 2100 50  0000 C CNN
-F 2 "" H 4150 1950 50  0001 C CNN
+F 2 "Capacitors_THT:C_Rect_L7.0mm_W2.5mm_P5.00mm" H 4150 1950 50  0001 C CNN
 F 3 "~" H 4150 1950 50  0001 C CNN
 	1    4150 1950
@@
 Connection ~ 4000 1950
 $Comp
-L Device:C_Small C7
+L device:C_Small C7
 U 1 1 5ADB6193
 P 2750 2100
 F 0 "C7" V 2850 2000 50  0000 C CNN
 F 1 "100n" V 2650 2100 50  0000 C CNN
-F 2 "" H 2750 2100 50  0001 C CNN
+F 2 "Capacitors_THT:C_Rect_L7.0mm_W2.5mm_P5.00mm" H 2750 2100 50  0001 C CNN
 F 3 "~" H 2750 2100 50  0001 C CNN
 	1    2750 2100
@@
 Connection ~ 1900 1900
 $Comp
-L Device:POT RV1
+L device:POT RV1
 U 1 1 5ADEF31B
 P 1900 2550
 F 0 "RV1" H 2100 2450 50  0000 R CNN
 F 1 "2k" V 1900 2600 50  0000 R CNN
-F 2 "" H 1900 2550 50  0001 C CNN
+F 2 "Potentiometers:Potentiometer_Trimmer_Bourns_3296X" H 1900 2550 50  0001 C CNN
 F 3 "~" H 1900 2550 50  0001 C CNN
 	1    1900 2550
@@
 F 0 "P3" H 3250 2600 50  0000 L CNN
 F 1 "CONTROL_IN" V 3400 2650 50  0000 L CNN
-F 2 "" H 3250 2900 50  0000 C CNN
+F 2 "w_conn_kk100:kk100_22-23-2051" H 3250 2900 50  0001 C CNN
 F 3 "" H 3250 2900 50  0000 C CNN
 	1    3250 2900
@@
 $EndComp
 $Comp
-L device:ZENERsmall D6
+L V_AMP-rescue:device_ZENERsmall-V_AMP-cache D6
 U 1 1 5AFB8EA2
 P 2450 1400
 F 0 "D6" H 2350 1450 50  0000 C CNN
 F 1 "5V1" H 2550 1450 50  0000 C CNN
-F 2 "" H 2450 1400 50  0000 C CNN
+F 2 "Diodes_THT:D_DO-41_SOD81_P7.62mm_Horizontal" H 2450 1400 50  0001 C CNN
 F 3 "" H 2450 1400 50  0000 C CNN
 	1    2450 1400
@@
 P 2650 1200
 F 0 "P2" H 2751 1176 50  0000 L CNN
-F 1 "BNC" H 2751 1085 50  0000 L CNN
-F 2 "" H 2650 1200 50  0000 C CNN
+F 1 "OUTPUT" H 2751 1085 50  0000 L CNN
+F 2 "Connect:bornier2" H 2650 1200 50  0001 C CNN
 F 3 "" H 2650 1200 50  0000 C CNN
 	1    2650 1200
