File: Circuits/P_SUPPLY/P_SUPPLY.sch (KiCad schematic (older format))
At the start: 28 parts, among them P1 127VAC, P2 ON/OFF SW, P3 SYMMETRIC 8V OUT, P4 +5V OUTPUT, T1 127:12, U1 LM7808CT, U2 LM7805CT, U3 LM7908CT

Commit message: ADD: Holes in Power Supply PCB
Changed lines of the file:
@@
 encoding utf-8
 Sheet 1 1
-Title "ELECTRIC KETTLE CIRCUIT"
-Date "2017-12-17"
-Rev ""
-Comp "FEDERAL UNIVERSITY OF RIO GRANDE DO SUL"
-Comment1 "Gabriel Luis"
-Comment2 "Lucas Sessegolo"
-Comment3 "Alisson Claudino"
-Comment4 "Designed by:"
+Title "SADAMAP POWER SUPPLY"
+Date "2018-01-31"
+Rev "2"
+Comp "LAPMA/CTA - IF/UFRGS"
+Comment1 "All resistors are 1/4W"
+Comment2 "The transformer 12+12 should have 800mA minimum current"
+Comment3 "Designed by: Alisson Claudino"
+Comment4 ""
 $EndDescr
 $Comp
@@
 F 0 "U1" H 1350 2900 50  0000 C CNN
 F 1 "LM7808CT" H 1450 2900 50  0000 L CNN
-F 2 "Power_Integrations:TO-220" H 1550 2800 50  0000 C CIN
+F 2 "Power_Integrations:TO-220" H 1550 2800 50  0001 C CIN
 F 3 "" H 1550 2700 50  0000 C CNN
 	1    1550 2700
@@
 F 0 "U3" H 3350 2500 50  0000 C CNN
 F 1 "LM7908CT" H 3450 2500 50  0000 L CNN
-F 2 "Power_Integrations:TO-220" H 3550 2600 50  0000 C CIN
+F 2 "Power_Integrations:TO-220" H 3550 2600 50  0001 C CIN
 F 3 "" H 3550 2700 50  0000 C CNN
 	1    3550 2700

Commit message: EDIT: REORGANIZING FILES
Parts:
- C1, C2, C3, C4, C5, C6, C7: symbol CP -> P_SUPPLY-rescue:CP
- D1, D2, D7: symbol Led_Small -> P_SUPPLY-rescue:Led_Small
- D3, D4, D5, D6: symbol D_Small -> P_SUPPLY-rescue:D_Small
- F1, F2, F3: symbol F_Small -> P_SUPPLY-rescue:F_Small
- P1, P2, P4: symbol CONN_01X02 -> P_SUPPLY-rescue:CONN_01X02
- P3: symbol CONN_01X03 -> P_SUPPLY-rescue:CONN_01X03
- R1, R2, R3: symbol R -> P_SUPPLY-rescue:R
- T1: symbol TRANSFO4 -> P_SUPPLY-rescue:TRANSFO4
- U1: symbol LM7808CT -> P_SUPPLY-rescue:LM7808CT
- U2: symbol LM7805CT -> P_SUPPLY-rescue:LM7805CT
- U3: symbol LM7908CT -> P_SUPPLY-rescue:LM7908CT
