File: Circuits/TEMP_MODULE/TEMP_MODULE.sch (KiCad schematic (older format))
At the start: 2 parts, among them J1 MAX31856_ThermoCouple_Module, P1 MCU_IN

Commit message: EDIT: REORGANIZING FILES
Parts:
- J1: symbol MAX31856_ThermoCouple_Module -> TEMP_MODULE-rescue:MAX31856_ThermoCouple_Module
- P1: symbol CONN_01X06 -> TEMP_MODULE-rescue:CONN_01X06
Changed lines of the file:
@@
-EESchema Schematic File Version 2
-LIBS:74xgxx
-LIBS:74xx
-LIBS:ac-dc
-LIBS:actel
-LIBS:adc-dac
-LIBS:Altera
-LIBS:analog_devices
-LIBS:analog_switches
-LIBS:atmel
-LIBS:audio
-LIBS:brooktre
-LIBS:cmos4000
-LIBS:cmos_ieee
-LIBS:conn
-LIBS:contrib
-LIBS:cypress
-LIBS:dc-dc
-LIBS:device
-LIBS:digital-audio
-LIBS:diode
-LIBS:display
-LIBS:dsp
-LIBS:elec-unifil
-LIBS:ESD_Protection
-LIBS:ftdi
-LIBS:gennum
-LIBS:graphic
-LIBS:hc11
-LIBS:intel
-LIBS:interface
-LIBS:ir
-LIBS:Lattice
-LIBS:linear
-LIBS:logo
-LIBS:maxim
-LIBS:memory
-LIBS:microchip
-LIBS:microchip_dspic33dsc
-LIBS:microchip_pic10mcu
-LIBS:microchip_pic12mcu
-LIBS:microchip_pic16mcu
-LIBS:microchip_pic18mcu
-LIBS:microchip_pic32mcu
-LIBS:microcontrollers
-LIBS:motor_drivers
-LIBS:motorola
-LIBS:msp430
-LIBS:nordicsemi
-LIBS:nxp_armmcu
-LIBS:onsemi
-LIBS:opto
-LIBS:Oscillators
-LIBS:philips
-LIBS:power
-LIBS:powerint
-LIBS:Power_Management
-LIBS:references
-LIBS:regul
-LIBS:relays
-LIBS:rfcom
-LIBS:sensors
-LIBS:silabs
-LIBS:siliconi
-LIBS:stm8
-LIBS:stm32
-LIBS:supertex
-LIBS:switches
-LIBS:texas
-LIBS:transf
-LIBS:transistors
-LIBS:ttl_ieee
-LIBS:valves
-LIBS:video
-LIBS:w_analog
-LIBS:w_connectors
-LIBS:w_device
-LIBS:w_logic
-LIBS:w_memory
-LIBS:w_microcontrollers
-LIBS:w_opto
-LIBS:Worldsemi
-LIBS:w_relay
-LIBS:w_rtx
-LIBS:w_transistor
-LIBS:w_vacuum
-LIBS:Xicor
-LIBS:xilinx
-LIBS:Zilog
+EESchema Schematic File Version 4
 LIBS:TEMP_MODULE-cache
-EELAYER 25 0
+EELAYER 26 0
 EELAYER END
 $Descr A4 11693 8268
@@
 $EndDescr
 $Comp
-L MAX31856_ThermoCouple_Module J1
+L TEMP_MODULE-rescue:MAX31856_ThermoCouple_Module J1
 U 1 1 5A9D6132
 P 6350 4125
@@
 ~CS
 $Comp
-L +5V #PWR01
+L TEMP_MODULE-rescue:+5V #PWR01
 U 1 1 5A9EE8DA
 P 6700 3725
@@
 $EndComp
 $Comp
-L GND #PWR02
+L TEMP_MODULE-rescue:GND #PWR02
 U 1 1 5A9EE90A
 P 6700 3525
@@
 $EndComp
 $Comp
-L GND #PWR03
+L TEMP_MODULE-rescue:GND #PWR03
 U 1 1 5A9EE97C
 P 6000 3725
@@
 SCK
 $Comp
-L CONN_01X06 P1
+L TEMP_MODULE-rescue:CONN_01X06 P1
 U 1 1 5A9EE9E7
 P 5175 4025
@@
 $EndComp
 $Comp
-L GND #PWR04
+L TEMP_MODULE-rescue:GND #PWR04
 U 1 1 5A9EEA44
 P 5375 4275
@@
 $EndComp
 $Comp
-L +5V #PWR05
+L TEMP_MODULE-rescue:+5V #PWR05
 U 1 1 5A9EEA6F
 P 5375 4175
@@
 NoConn ~ 6700 3425
 $Comp
-L GND #PWR06
+L TEMP_MODULE-rescue:GND #PWR06
 U 1 1 5AA07283
 P 5350 4750
@@
 $EndComp
 $Comp
-L +5V #PWR07
+L TEMP_MODULE-rescue:+5V #PWR07
 U 1 1 5AA07289
 P 5350 4650
@@
 $EndComp
 $Comp
-L PWR_FLAG #FLG08
+L TEMP_MODULE-rescue:PWR_FLAG #FLG08
 U 1 1 5AA0729B
 P 5300 4625
@@
 $EndComp
 $Comp
-L PWR_FLAG #FLG09
+L TEMP_MODULE-rescue:PWR_FLAG #FLG09
 U 1 1 5AA072B3
 P 5300 4800
