File: Circuits/ADC_MCU_MODULE/ADC_MCU_MODULE.sch (KiCad schematic (older format))
At the start: 30 parts, among them J1 Arduino_Nano_Header, P1 POWER, P2 BNC, P3 BNC, P4 BNC, P5 BNC, P6 BNC, P7 BNC, P8 BNC, P9 BNC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

Commit message: ADD: ADC/MCU Module Fabrication Files
Parts:
- added P10: TEMP_MODULE_OUT, w_conn_kk156:kk156_26-60-4060, symbol CONN_01X06
Connections:
- net +5V: now also P10.2 (P2)
- net GND: now also P10.1 (P1)
- net ~CS: now reaches J1.11 (D8/ICP)
- net ~CS: now also P10.3 (P3)
- net MOSI: now reaches J1.14 (D11/MOSI)
- net MOSI: now also P10.5 (P5)
- net MISO: now reaches J1.15 (D12/MISO)
- net MISO: now also P10.4 (P4)
- net SCK: now reaches J1.16 (SCK/D13)
- net SCK: now also P10.6 (P6)
- no-connect marks 26 -> 22
Other:
- note added: "MAX31856 Temperature Module Header"
Changed lines of the file:
@@
 Wire Notes Line
 	8000 2725 8000 5300
-NoConn ~ 9250 4400
 NoConn ~ 9250 4200
 NoConn ~ 9250 3500
@@
 NoConn ~ 8550 3800
 NoConn ~ 8550 3900
-NoConn ~ 8550 4000
 NoConn ~ 8550 4100
 NoConn ~ 8550 4200
-NoConn ~ 8550 4300
-NoConn ~ 8550 4400
 NoConn ~ 9250 3800
 NoConn ~ 9250 3900
@@
 NoConn ~ 9250 4300
 $Comp
-L GND #PWR?
+L GND #PWR020
 U 1 1 5A974874
 P 8425 3350
-F 0 "#PWR?" H 8425 3100 50  0001 C CNN
+F 0 "#PWR020" H 8425 3100 50  0001 C CNN
 F 1 "GND" H 8425 3200 50  0000 C CNN
 F 2 "" H 8425 3350 50  0000 C CNN
@@
 Wire Wire Line
 	8425 3300 8550 3300
+Text GLabel 9250 4400 2    47   BiDi ~ 0
+SCK
+Text GLabel 8550 4400 0    47   Input ~ 0
+MISO
+Text GLabel 8550 4300 0    47   Output ~ 0
+MOSI
+Text GLabel 8550 4000 0    47   Output ~ 0
+~CS
+$Comp
+L CONN_01X06 P10
+U 1 1 5AA06AB3
+P 6975 3300
+F 0 "P10" H 6975 3650 50  0001 C CNN
+F 1 "TEMP_MODULE_OUT" V 7075 3300 50  0000 C CNN
+F 2 "w_conn_kk156:kk156_26-60-4060" H 6975 3300 50  0001 C CNN
+F 3 "" H 6975 3300 50  0000 C CNN
+	1    6975 3300
+	-1   0    0    1
+$EndComp
+$Comp
+L GND #PWR021
+U 1 1 5AA06B80
+P 7175 3550
+F 0 "#PWR021" H 7175 3300 50  0001 C CNN
+F 1 "GND" V 7175 3375 50  0000 C CNN
+F 2 "" H 7175 3550 50  0000 C CNN
+F 3 "" H 7175 3550 50  0000 C CNN
+	1    7175 3550
+	0    -1   -1   0
+$EndComp
+$Comp
+L +5V #PWR022
+U 1 1 5AA06CD4
+P 7175 3450
+F 0 "#PWR022" H 7175 3300 50  0001 C CNN
+F 1 "+5V" V 7175 3625 50  0000 C CNN
+F 2 "" H 7175 3450 50  0000 C CNN
+F 3 "" H 7175 3450 50  0000 C CNN
+	1    7175 3450
+	0    1    1    0
+$EndComp
+Text GLabel 7175 3350 2    47   Input ~ 0
+~CS
+Text GLabel 7175 3150 2    47   Input ~ 0
+MOSI
+Text GLabel 7175 3250 2    47   Output ~ 0
+MISO
+Text GLabel 7175 3050 2    47   BiDi ~ 0
+SCK
+Text Notes 6500 3775 0    47   ~ 0
+MAX31856 Temperature Module Header
+Wire Notes Line
+	7950 2925 7950 3800
+Wire Notes Line
+	7950 3800 6475 3800
+Wire Notes Line
+	6475 3800 6475 2925
+Wire Notes Line
+	6475 2925 7950 2925
 $EndSCHEMATC

Commit message: EDIT: REORGANIZING FILES
Parts:
- C1: symbol CP_Small -> ADC_MCU_MODULE-rescue:CP_Small
- C2, C3, C4, C5, C6, C7, C8, C9: symbol C_Small -> ADC_MCU_MODULE-rescue:C_Small
- J1: symbol Arduino_Nano_Header -> ADC_MCU_MODULE-rescue:Arduino_Nano_Header
- P1: symbol CONN_01X02 -> ADC_MCU_MODULE-rescue:CONN_01X02
- P10: symbol CONN_01X06 -> ADC_MCU_MODULE-rescue:CONN_01X06
- P2, P3, P4, P5, P6, P7, P8, P9: symbol BNC -> ADC_MCU_MODULE-rescue:BNC
- R1, R2, R3, R4, R5, R6, R7, R8, R9: symbol R -> ADC_MCU_MODULE-rescue:R
- U1, U2: symbol ADS1115 -> ADC_MCU_MODULE-rescue:ADS1115

Commit message: EDIT: ADC_MCU new schematic
Parts:
- added P11: V_AMP_1, w_conn_kk156:kk156_26-64-4050, symbol conn:CONN_01X05
- added P12: V_AMP_2, w_conn_kk156:kk156_26-64-4050, symbol conn:CONN_01X05
- added P13: V_AMP_3, w_conn_kk156:kk156_26-64-4050, symbol conn:CONN_01X05
Connections:
- net labels added: V1_b0, V1_b1, V1_b2, V1_b3, V2_b0, V2_b1, V2_b2, V2_b3, V3_b0, V3_b1, V3_b2, V3_b3
- wire segments 81 -> 79
- no-connect marks 22 -> 10
Other:
- note added: "Voltage Amplifier Gain Control - 1 to 3"
Changed lines of the file:
@@
 NoConn ~ 8550 3100
 NoConn ~ 8550 3000
-NoConn ~ 8550 3400
-NoConn ~ 8550 3500
-NoConn ~ 8550 3600
-NoConn ~ 8550 3700
-NoConn ~ 8550 3800
-NoConn ~ 8550 3900
-NoConn ~ 8550 4100
-NoConn ~ 8550 4200
-NoConn ~ 9250 3800
-NoConn ~ 9250 3900
-NoConn ~ 9250 4000
-NoConn ~ 9250 4100
 NoConn ~ 9250 4300
-$Comp
-L ADC_MCU_MODULE-rescue:GND #PWR020
-U 1 1 5A974874
-P 8425 3350
-F 0 "#PWR020" H 8425 3100 50  0001 C CNN
-F 1 "GND" H 8425 3200 50  0000 C CNN
-F 2 "" H 8425 3350 50  0000 C CNN
-F 3 "" H 8425 3350 50  0000 C CNN
-	1    8425 3350
-	1    0    0    -1
-$EndComp
-Wire Wire Line
-	8425 3350 8425 3300
-Wire Wire Line
-	8425 3300 8550 3300
 Text GLabel 9250 4400 2    47   BiDi ~ 0
 SCK
@@
 Text GLabel 8550 4300 0    47   Output ~ 0
 MOSI
-Text GLabel 8550 4000 0    47   Output ~ 0
+Text GLabel 8550 4000 0    39   Output ~ 0
 ~CS
 $Comp
@@
 Wire Wire Line
 	2175 2925 2225 2925
+Text GLabel 9250 4100 2    50   Input ~ 0
+V1_b0
+Text GLabel 9250 4000 2    50   Input ~ 0
+V1_b1
+Text GLabel 9250 3900 2    50   Input ~ 0
+V1_b2
+Text GLabel 9250 3800 2    50   Input ~ 0
+V1_b3
+Text GLabel 8550 4200 0    47   Input ~ 0
+V2_b0
+Text GLabel 8550 4100 0    47   Input ~ 0
+V2_b1
+Text GLabel 8550 3900 0    47   Input ~ 0
+V2_b2
+Text GLabel 8550 3800 0    47   Input ~ 0
+V2_b3
+Text GLabel 8550 3700 0    47   Input ~ 0
+V3_b0
+Text GLabel 8550 3600 0    47   Input ~ 0
+V3_b1
+$Comp
+L ADC_MCU_MODULE-rescue:GND #PWR020
+U 1 1 5A974874
+P 8550 3300
+F 0 "#PWR020" H 8550 3050 50  0001 C CNN
+F 1 "GND" V 8550 3100 50  0000 C CNN
+F 2 "" H 8550 3300 50  0000 C CNN
+F 3 "" H 8550 3300 50  0000 C CNN
+	1    8550 3300
+	0    1    1    0
+$EndComp
+Text GLabel 8550 3500 0    47   Input ~ 0
+V3_b2
+Text GLabel 8550 3400 0    47   Input ~ 0
+V3_b3
+$Comp
+L conn:CONN_01X05 P13
+U 1 1 5B2A908C
+P 5800 2850
+F 0 "P13" V 5765 2562 50  0000 R CNN
+F 1 "V_AMP_3" V 5900 3000 50  0000 R CNN
+F 2 "w_conn_kk156:kk156_26-64-4050" H 5800 2850 50  0001 C CNN
+F 3 "" H 5800 2850 50  0000 C CNN
+	1    5800 2850
+	0    -1   -1   0
+$EndComp
+Text GLabel 5700 3050 3    47   Input ~ 0
+V3_b3
+$Comp
+L ADC_MCU_MODULE-rescue:GND #PWR0101
+U 1 1 5B2A93F4
+P 5600 3050
+F 0 "#PWR0101" H 5600 2800 50  0001 C CNN
+F 1 "GND" V 5605 2877 50  0000 C CNN
+F 2 "" H 5600 3050 50  0000 C CNN
+F 3 "" H 5600 3050 50  0000 C CNN
+	1    5600 3050
+	1    0    0    -1
+$EndComp
+Text GLabel 5800 3050 3    47   Input ~ 0
+V3_b2
+Text GLabel 5900 3050 3    47   Input ~ 0
+V3_b1
+Text GLabel 6000 3050 3    47   Input ~ 0
+V3_b0
+$Comp
+L conn:CONN_01X05 P12
+U 1 1 5B2AB538
+P 5050 2850
+F 0 "P12" V 5015 2562 50  0000 R CNN
+F 1 "V_AMP_2" V 5150 3000 50  0000 R CNN
+F 2 "w_conn_kk156:kk156_26-64-4050" H 5050 2850 50  0001 C CNN
+F 3 "" H 5050 2850 50  0000 C CNN
+	1    5050 2850
+	0    -1   -1   0
+$EndComp
+Text GLabel 4950 3050 3    47   Input ~ 0
+V2_b3
+$Comp
+L ADC_MCU_MODULE-rescue:GND #PWR0102
+U 1 1 5B2AB540
+P 4850 3050
+F 0 "#PWR0102" H 4850 2800 50  0001 C CNN
+F 1 "GND" V 4855 2877 50  0000 C CNN
+F 2 "" H 4850 3050 50  0000 C CNN
+F 3 "" H 4850 3050 50  0000 C CNN
+	1    4850 3050
+	1    0    0    -1
+$EndComp
+Text GLabel 5050 3050 3    47   Input ~ 0
+V2_b2
+Text GLabel 5150 3050 3    47   Input ~ 0
+V2_b1
+Text GLabel 5250 3050 3    47   Input ~ 0
+V2_b0
+$Comp
+L conn:CONN_01X05 P11
+U 1 1 5B2AD87C
+P 4300 2850
+F 0 "P11" V 4265 2562 50  0000 R CNN
+F 1 "V_AMP_1" V 4400 3000 50  0000 R CNN
+F 2 "w_conn_kk156:kk156_26-64-4050" H 4300 2850 50  0001 C CNN
+F 3 "" H 4300 2850 50  0000 C CNN
+	1    4300 2850
+	0    -1   -1   0
+$EndComp
+Text GLabel 4200 3050 3    47   Input ~ 0
+V1_b3
+$Comp
+L ADC_MCU_MODULE-rescue:GND #PWR0103
+U 1 1 5B2AD884
+P 4100 3050
+F 0 "#PWR0103" H 4100 2800 50  0001 C CNN
+F 1 "GND" V 4105 2877 50  0000 C CNN
+F 2 "" H 4100 3050 50  0000 C CNN
+F 3 "" H 4100 3050 50  0000 C CNN
+	1    4100 3050
+	1    0    0    -1
+$EndComp
+Text GLabel 4300 3050 3    47   Input ~ 0
+V1_b2
+Text GLabel 4400 3050 3    47   Input ~ 0
+V1_b1
+Text GLabel 4500 3050 3    47   Input ~ 0
+V1_b0
+Text Notes 4250 3450 0    50   ~ 0
+Voltage Amplifier Gain Control - 1 to 3
+Wire Notes Line
+	3950 2650 6200 2650
+Wire Notes Line
+	6200 2650 6200 3500
+Wire Notes Line
+	6200 3500 3950 3500
+Wire Notes Line
+	3950 2650 3950 3500
 $EndSCHEMATC

Commit message: ADD: ADC_MCU New Schematic
Parts:
- C1: footprint Capacitors_THT:CP_Radial_D5.0mm_P2.50mm -> Capacitors_ThroughHole:C_Radial_D5_L6_P2.5
- C2, C3, C4, C5, C6, C7, C8, C9: footprint Capacitors_THT:C_Rect_L7.0mm_W2.5mm_P5.00mm -> Capacitors_ThroughHole:C_Rect_L7_W2.5_P5
- P10: footprint w_conn_kk156:kk156_26-60-4060 -> w_conn_kk100:kk100_22-23-2061
- P11: value V_AMP_1 -> V_AMP SEL CH-B; footprint w_conn_kk156:kk156_26-64-4050 -> w_conn_kk100:kk100_22-23-2051
- P12: value V_AMP_2 -> V_AMP SEL CH-A; footprint w_conn_kk156:kk156_26-64-4050 -> w_conn_kk100:kk100_22-23-2051
- P13: value V_AMP_3 -> V_AMP SEL CH-C; footprint w_conn_kk156:kk156_26-64-4050 -> w_conn_kk100:kk100_22-23-2051
- P2, P3, P4, P5, P6, P7, P8, P9: footprint Connectors:bnc-ci -> Connectors:bornier2
- U1, U2: footprint w_pin_strip:pin_socket_10 -> Misc:ADS1115
Connections:
- net labels added: VA0, VA1, VA2, VA3, VB0, VB1, VB2, VB3, VC0, VC1, VC2, VC3
- net labels removed: V1_b0, V1_b1, V1_b2, V1_b3, V2_b0, V2_b1, V2_b2, V2_b3, V3_b0, V3_b1, V3_b2, V3_b3
- wire segments 79 -> 87
Other:
- note added: "Digital Voltage Amplifier Controls"
- note removed: "Voltage Amplifier Gain Control - 1 to 3"
